File: Fan Speed Controller.kicad_pcb (KiCad board)
At the start: 2 copper layers, 11 parts, among them IC1 LM555CMMX_NOPB, J1 22-23-2031, J2 163-179PH-EX, J3 22-23-2031, J4 22-23-2031, J5 22-23-2031, Q1 ZXMN3A01FTA

Commit message: Completed V1 of circuit/board
Parts:
- added C1: C0.1uf, Capacitor_THT:C_Axial_L3.8mm_D2.6mm_P10.00mm_Horizontal, F.Cu at (65.4, 70.9)
- added C2: C10nf, Capacitor_THT:C_Disc_D5.0mm_W2.5mm_P5.00mm, F.Cu at (75.4, 59.7)
- added R1: R1k, Resistor_THT:R_Axial_DIN0207_L6.3mm_D2.5mm_P10.16mm_Horizontal, F.Cu at (59.9, 44.4)
- added R2: R1k, Resistor_THT:R_Axial_DIN0207_L6.3mm_D2.5mm_P10.16mm_Horizontal, F.Cu at (54.6, 44.4)
- added R3: R1k, Resistor_THT:R_Axial_DIN0207_L6.3mm_D2.5mm_P10.16mm_Horizontal, F.Cu at (65.5, 54.6)
- added S1: SLW-883935-2A-D, Library:SLW8839352AD, F.Cu at (43.4, 51.5)
- moved J1 53.9 mm to (41.9, 33.5), turned to 0 degrees
- moved J2 51.1 mm to (54.9, 33.5)
- moved D1 43.3 mm to (72.1, 44.7), turned to -90 degrees
- moved R4 41.0 mm to (87.7, 65.0), turned to 180 degrees
- moved D3 40.1 mm to (77.2, 44.4), turned to -90 degrees
- moved J3 39.7 mm to (67.8, 33.5)
- moved J5 34.2 mm to (50.4, 65.0)
- moved J4 31.5 mm to (80.8, 33.5)
- moved D2 31.2 mm to (83.6, 52.0), turned to 90 degrees
- moved Q1 23.1 mm to (70.4, 63.5), turned to 90 degrees
- moved IC1 22.9 mm to (64.0, 62.5), turned to 90 degrees
- renumbered J3 to J2, J4 to J3, J5 to J4, J2 to J5
Connections:
- D2 pad 1: unconnected-(D2-K-Pad1) -> Net-(D2-K)
- D2 pad 2: unconnected-(D2-A-Pad2) -> Net-(D2-A)
- D3 pad 1: unconnected-(D3-K-Pad1) -> Net-(D2-A)
- D3 pad 2: unconnected-(D3-A-Pad2) -> Net-(D3-A)
- IC1 pad 2: unconnected-(IC1-TRIGGER-Pad2) -> GND
- IC1 pad 4: unconnected-(IC1-RESET-Pad4) -> +12V
- IC1 pad 5: unconnected-(IC1-CONTROL_VOLTAGE-Pad5) -> Net-(IC1-CONTROL_VOLTAGE)
- IC1 pad 6: unconnected-(IC1-THRESHOLD-Pad6) -> GND
- IC1 pad 7: unconnected-(IC1-DISCHARGE-Pad7) -> Net-(D2-A)
- J1 pad 1: Net-(D1-A) -> GND
- J1 pad 3: Net-(D1-A) -> GND
- J2 pad 1: Net-(D1-A) -> GND
- J2 pad 3: Net-(D1-A) -> GND
- J3 pad 1: Net-(D1-A) -> GND
- J3 pad 3: Net-(D1-A) -> GND
- J4 pad 1: Net-(D1-A) -> GND
- J4 pad 3: Net-(D1-A) -> GND
- J5 pad A: +12V -> Net-(S1-COM)
- R4 pad 1: unconnected-(R4-Pad1) -> Net-(D2-K)
- R4 pad 2: unconnected-(R4-Pad2) -> Net-(C2-Pad1)
- R4 pad 3: unconnected-(R4-Pad3) -> Net-(D3-A)
Routing:
- net GND: track 0.00 -> 130.1 mm
- net +12V: track 0.00 -> 98.8 mm
- net Net-(D2-A): track 0.00 -> 28.7 mm
- net Net-(IC1-OUTPUT): track 0.00 -> 28.3 mm
- net Net-(S1-COM): track 0.00 -> 19.7 mm
- net Net-(Q1-G): track 0.00 -> 19.1 mm
- net Net-(C2-Pad1): track 0.00 -> 13.2 mm
- net Net-(IC1-CONTROL_VOLTAGE): track 0.00 -> 11.4 mm
- net Net-(D3-A): track 0.00 -> 11.3 mm
- net Net-(D2-K): track 0.00 -> 10.1 mm
- net Net-(D1-A): track 0.00 -> 8.36 mm
Other:
- board outline added: 57.1 x 44.5 mm
- board text added: "MIN POWER SUPPLY: 12V 1.5A FAN MAX: 4 DATE: MARCH 2024"
